File: panel_rp2354_20x20_v0p1/panel_header.kicad_sch (KiCad schematic)
At the start: 4 parts, among them J2 Conn_01x05, J3 Conn_01x05, J4 Conn_01x05, J5 Conn_01x05

Commit message: Fix most warnings
Other:
- company: (none) -> Janelia Research Campus
- title: (none) -> G6 Panel
Changed lines of the file:
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@@
 	(generator_version "9.0")
 	(paper "A4")
+	(title_block
+		(title "G6 Panel")
+		(date "2026-04-01")
+		(rev "0.1.3")
+		(company "Janelia Research Campus")
+	)
 	(text "1x5 Pin Header\n\nJLCPCB/LCSC\nPN C7296801\n\nDigikey PN: 952-M20-8890545RCT-ND\nManufacturer PN: M20-8890545R\n\nDigikey PN: 952-3266-ND\nManufacturer PN: M20-8900505"
 		(exclude_from_sim no)
@@
 		)
 		(instances
-			(project "driver_rp2350"
+			(project "panel_rp2354_20x20"
 				(path "/1e634561-32a0-4ffa-9d4f-e93f355464d5/35cc1d84-fe4a-4d4c-89d0-5c31c9afaae5"
 					(reference "#PWR0124")
@@
 		)
 		(instances
-			(project "driver_rp2350"
+			(project "panel_rp2354_20x20"
 				(path "/1e634561-32a0-4ffa-9d4f-e93f355464d5/35cc1d84-fe4a-4d4c-89d0-5c31c9afaae5"
 					(reference "#PWR0122")
@@
 		)
 		(instances
-			(project "driver_rp2350"
+			(project "panel_rp2354_20x20"
 				(path "/1e634561-32a0-4ffa-9d4f-e93f355464d5/35cc1d84-fe4a-4d4c-89d0-5c31c9afaae5"
 					(reference "#PWR0123")
@@
 		)
 		(instances
-			(project "driver_rp2350"
+			(project "panel_rp2354_20x20"
 				(path "/1e634561-32a0-4ffa-9d4f-e93f355464d5/35cc1d84-fe4a-4d4c-89d0-5c31c9afaae5"
 					(reference "J5")
@@
 		)
 		(instances
-			(project "driver_rp2350"
+			(project "panel_rp2354_20x20"
 				(path "/1e634561-32a0-4ffa-9d4f-e93f355464d5/35cc1d84-fe4a-4d4c-89d0-5c31c9afaae5"
 					(reference "J2")
@@
 		)
 		(instances
-			(project "driver_rp2350"
+			(project "panel_rp2354_20x20"
 				(path "/1e634561-32a0-4ffa-9d4f-e93f355464d5/35cc1d84-fe4a-4d4c-89d0-5c31c9afaae5"
 					(reference "J4")
@@
 		)
 		(instances
-			(project "driver_rp2350"
+			(project "panel_rp2354_20x20"
 				(path "/1e634561-32a0-4ffa-9d4f-e93f355464d5/35cc1d84-fe4a-4d4c-89d0-5c31c9afaae5"
 					(reference "J3")
