File: panel_rp2354_20x20_v0p1/panel_led.kicad_sch (KiCad schematic)
At the start: 420 parts

Commit message: Fix most warnings
Parts:
- R10, R11, R12, R13, R14, R15, R16, R17, R18, R19, R20, R21, R22, R23, R24, R25, R26, R27, R28, R9: footprint Resistor_SMD:R_0201_0603Metric -> panel_custom:R_0201_0603Metric
Other:
- company: (none) -> Janelia Research Campus
- title: (none) -> G6 Panel
