File: panel_rp2354_20x20_v0p1/panel_rp2354_20x20.kicad_sch (KiCad schematic)
At the start: 0 parts

Commit message: Fix most warnings
Other:
- company: (none) -> Janelia Research Campus
- title: (none) -> G6 Panel
Changed lines of the file:
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@@
 	(paper "USLetter")
 	(title_block
-		(date "9 may 2016")
+		(title "G6 Panel")
+		(date "2026-04-01")
+		(rev "0.1.3")
+		(company "Janelia Research Campus")
 	)
 	(text "Column Pins"
