File: panel_rp2354_20x20_v0p1/panel_usb_power.kicad_sch (KiCad schematic)
At the start: 4 parts, among them J1 Conn_01x04, U43 AP2112K-3.3

Commit message: Fix most warnings
Parts:
- C67, C68: footprint Capacitor_SMD:C_0402_1005Metric -> panel_custom:C_0402_1005Metric
- U43: footprint Package_TO_SOT_SMD:SOT-23-5 -> panel_custom:SOT-23-5; symbol Regulator_Linear:AP2112K-3.3 -> panel_custom:AP2112K-3.3
Other:
- company: (none) -> Janelia Research Campus
- title: (none) -> G6 Panel
Changed lines of the file:
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@@
 	(generator_version "9.0")
 	(paper "A4")
+	(title_block
+		(title "G6 Panel")
+		(date "2026-04-01")
+		(rev "0.1.3")
+		(company "Janelia Research Campus")
+	)
 	(text "3.3V Regulator"
 		(exclude_from_sim no)
@@
 		)
 		(instances
-			(project "driver_rp2350"
+			(project "panel_rp2354_20x20"
 				(path "/1e634561-32a0-4ffa-9d4f-e93f355464d5/e614504e-e15b-412a-a899-de4ba0827a39"
 					(reference "#PWR0118")
@@
 		)
 		(instances
-			(project "driver_rp2350"
+			(project "panel_rp2354_20x20"
 				(path "/1e634561-32a0-4ffa-9d4f-e93f355464d5/e614504e-e15b-412a-a899-de4ba0827a39"
 					(reference "#PWR0121")
@@
 		)
 		(instances
-			(project "driver_rp2350"
+			(project "panel_rp2354_20x20"
 				(path "/1e634561-32a0-4ffa-9d4f-e93f355464d5/e614504e-e15b-412a-a899-de4ba0827a39"
 					(reference "#PWR0117")
@@
 		)
 		(instances
-			(project ""
+			(project "panel_rp2354_20x20"
 				(path "/1e634561-32a0-4ffa-9d4f-e93f355464d5/e614504e-e15b-412a-a899-de4ba0827a39"
 					(reference "#FLG02")
@@
 		)
 		(instances
-			(project "driver_rp2350"
+			(project "panel_rp2354_20x20"
 				(path "/1e634561-32a0-4ffa-9d4f-e93f355464d5/e614504e-e15b-412a-a899-de4ba0827a39"
 					(reference "#PWR0119")
@@
 			)
 		)
-		(property "Footprint" "Capacitor_SMD:C_0402_1005Metric"
+		(property "Footprint" "panel_custom:C_0402_1005Metric"
 			(at 201.6252 57.15 0)
 			(effects
@@
 		)
 		(instances
-			(project "driver_rp2350"
+			(project "panel_rp2354_20x20"
 				(path "/1e634561-32a0-4ffa-9d4f-e93f355464d5/e614504e-e15b-412a-a899-de4ba0827a39"
 					(reference "C67")
@@
 		)
 		(instances
-			(project "panel_rp2350_20x20"
+			(project "panel_rp2354_20x20"
 				(path "/1e634561-32a0-4ffa-9d4f-e93f355464d5/e614504e-e15b-412a-a899-de4ba0827a39"
 					(reference "#PWR01")
@@
 		)
 		(instances
-			(project "panel_rp2350_20x20"
+			(project "panel_rp2354_20x20"
 				(path "/1e634561-32a0-4ffa-9d4f-e93f355464d5/e614504e-e15b-412a-a899-de4ba0827a39"
 					(reference "#FLG01")
@@
 		)
 		(instances
-			(project "driver_rp2350"
+			(project "panel_rp2354_20x20"
 				(path "/1e634561-32a0-4ffa-9d4f-e93f355464d5/e614504e-e15b-412a-a899-de4ba0827a39"
 					(reference "J1")
@@
 			)
 		)
-		(property "Footprint" "Capacitor_SMD:C_0402_1005Metric"
+		(property "Footprint" "panel_custom:C_0402_1005Metric"
 			(at 227.0252 57.15 0)
 			(effects
@@
 		)
 		(instances
-			(project "driver_rp2350"
+			(project "panel_rp2354_20x20"
 				(path "/1e634561-32a0-4ffa-9d4f-e93f355464d5/e614504e-e15b-412a-a899-de4ba0827a39"
 					(reference "C68")
@@
 	)
 	(symbol
-		(lib_id "Regulator_Linear:AP2112K-3.3")
+		(lib_id "panel_custom:AP2112K-3.3")
 		(at 214.63 48.26 0)
 		(unit 1)
@@
 			)
 		)
-		(property "Footprint" "Package_TO_SOT_SMD:SOT-23-5"
+		(property "Footprint" "panel_custom:SOT-23-5"
 			(at 214.63 40.005 0)
 			(effects
@@
 		)
 		(instances
-			(project "driver_rp2350"
+			(project "panel_rp2354_20x20"
 				(path "/1e634561-32a0-4ffa-9d4f-e93f355464d5/e614504e-e15b-412a-a899-de4ba0827a39"
 					(reference "U43")
@@
 		)
 		(instances
-			(project "driver_rp2350"
+			(project "panel_rp2354_20x20"
 				(path "/1e634561-32a0-4ffa-9d4f-e93f355464d5/e614504e-e15b-412a-a899-de4ba0827a39"
 					(reference "#PWR0120")
@@
 		)
 		(instances
-			(project ""
+			(project "panel_rp2354_20x20"
 				(path "/1e634561-32a0-4ffa-9d4f-e93f355464d5/e614504e-e15b-412a-a899-de4ba0827a39"
 					(reference "#PWR02")

Commit message: Fixed ERC and DRC warnings and regenerated production files
Parts:
- C67: footprint panel_custom:C_0402_1005Metric -> panel_custom:C_0402_1005Metric_NoSilk
Changed lines of the file:
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@@
 			)
 		)
-		(property "Footprint" "panel_custom:C_0402_1005Metric"
+		(property "Footprint" "panel_custom:C_0402_1005Metric_NoSilk"
 			(at 201.6252 57.15 0)
 			(effects
