File: panel_rp2354_20x20_v0p1/manual_route/1st_layout/rev0/panel_rp2350_20x20_rev0.kicad_pcb (KiCad board)
At the start: 6 copper layers, 45 x 45 mm, 556 parts, among them J1 Conn_01x04, J2 Conn_01x05, J3 Conn_01x05, J4 Conn_01x05, J5 Conn_01x05, SW1 SW_Push, SW2 SW_Push, U1 APS6404L-3SQR, U10 UCC27517, U11 UCC27517, U12 UCC27517, U13 UCC27517, U14 UCC27517, U15 UCC27517, U16 UCC27517, U17 UCC27517, U18 UCC27517, U19 UCC27517, U2 RP2354B_80QFN, U20 UCC27517, U21 UCC27517, U22 UCC27517, U23 UCC27517, U24 UCC27517, U25 UCC27517, U26 UCC27517, U27 UCC27517, U28 UCC27517, U29 UCC27517, U3 UCC27517, U30 UCC27517, U31 UCC27517, U32 UCC27517, U33 UCC27517, U34 UCC27517, U35 UCC27517, U36 UCC27517, U37 UCC27517, U38 UCC27517, U39 UCC27517, U4 UCC27517, U40 UCC27517, U41 UCC27517, U42 UCC27517, U43 AP2112K-3.3, U5 UCC27517, U6 UCC27517, U7 UCC27517, U8 UCC27517, U9 UCC27517, Y1 ABM8-272-T3

Commit message: Fix most warnings
Parts:
- C4, C5: footprint RP2350_80QFN_minimal:C_0402_1005Metric_small_pads -> panel_custom:C_0402_1005Metric_small_pads
- L1: footprint RP2350_80QFN_minimal:L_pol_2016 -> panel_custom:L_pol_2016
- U2: footprint RP2350_80QFN_minimal:RP2350-QFN-80-1EP_10x10_P0.4mm_EP3.4x3.4mm_ThermalVias -> panel_custom:RP2350-QFN-80-1EP_10x10_P0.4mm_EP3.4x3.4mm_ThermalVias
Changed lines of the file:
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@@
 		)
 	)
-	(footprint "RP2350_80QFN_minimal:C_0402_1005Metric_small_pads"
+	(footprint "panel_custom:C_0402_1005Metric_small_pads"
 		(layer "B.Cu")
 		(at 75.5 82.4)
@@
 		)
 	)
-	(footprint "RP2350_80QFN_minimal:RP2350-QFN-80-1EP_10x10_P0.4mm_EP3.4x3.4mm_ThermalVias"
+	(footprint "panel_custom:RP2350-QFN-80-1EP_10x10_P0.4mm_EP3.4x3.4mm_ThermalVias"
 		(layer "B.Cu")
 		(at 72.5 76)
@@
 		)
 		(embedded_fonts no)
-		(model "${KIPRJMOD}/RP2350_80QFN_minimal.pretty/RP2350_QFN80.step"
+		(model "${KIPRJMOD}/panel_custom.pretty/RP2350_QFN80.step"
 			(offset
 				(xyz 0 0 0)
@@
 		)
 	)
-	(footprint "RP2350_80QFN_minimal:L_pol_2016"
+	(footprint "panel_custom:L_pol_2016"
 		(layer "B.Cu")
 		(at 75.5 85.025)
@@
 		)
 	)
-	(footprint "RP2350_80QFN_minimal:C_0402_1005Metric_small_pads"
+	(footprint "panel_custom:C_0402_1005Metric_small_pads"
 		(layer "B.Cu")
 		(at 75.44 83.375)
