File: panel_rp2354_20x20_v0p2/panel_mcu.kicad_sch (KiCad schematic)
At the start: 32 parts, among them SW1 SW_Push, SW2 SW_Push, U1 APS6404L-3SQR, U2 RP2354B_80QFN, Y1 ABM8-272-T3

Commit message: Consolidate v0p2 project libraries and clean generated files
Parts:
- C4, C5: footprint RP2350_80QFN_minimal:C_0402_1005Metric_small_pads -> panel_custom:C_0402_1005Metric_small_pads
- L1: footprint RP2350_80QFN_minimal:L_pol_2016 -> panel_custom:L_pol_2016
- U2: footprint RP2350_80QFN_minimal:RP2350-QFN-80-1EP_10x10_P0.4mm_EP3.4x3.4mm_ThermalVias -> panel_custom:RP2350-QFN-80-1EP_10x10_P0.4mm_EP3.4x3.4mm_ThermalVias
Changed lines of the file:
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@@
 			)
 		)
-		(property "Footprint" "RP2350_80QFN_minimal:RP2350-QFN-80-1EP_10x10_P0.4mm_EP3.4x3.4mm_ThermalVias"
+		(property "Footprint" "panel_custom:RP2350-QFN-80-1EP_10x10_P0.4mm_EP3.4x3.4mm_ThermalVias"
 			(at 185.42 115.57 0)
 			(effects
@@
 			)
 		)
-		(property "Footprint" "RP2350_80QFN_minimal:L_pol_2016"
+		(property "Footprint" "panel_custom:L_pol_2016"
 			(at 140.97 78.74 0)
 			(effects
@@
 			)
 		)
-		(property "Footprint" "RP2350_80QFN_minimal:C_0402_1005Metric_small_pads"
+		(property "Footprint" "panel_custom:C_0402_1005Metric_small_pads"
 			(at 126.6952 82.55 0)
 			(effects
@@
 			)
 		)
-		(property "Footprint" "RP2350_80QFN_minimal:C_0402_1005Metric_small_pads"
+		(property "Footprint" "panel_custom:C_0402_1005Metric_small_pads"
 			(at 115.2652 82.55 0)
 			(effects
